Commit message: tmp disable grip f3 collision.

File: mycobot_description/urdf/mycobot/mycobot_with_gripper_up.urdf (robot description, URDF)
Before this commit: robot firefighter, 15 links, 14 joints
Links:
- link gripper_left3: geometry visual mesh filename=package://mycobot_description/urdf/mycobot/gripper_left3.dae
- link gripper_right3: geometry visual mesh filename=package://mycobot_description/urdf/mycobot/gripper_right3.d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
